Commit message: Changes in according to gsilano/Bebops#8

File: rotors_description/urdf/component_snippets.xacro (robot description, xacro)
@@ -17,5 +17,4 @@
 -->
 <robot xmlns:xacro="http://ros.org/wiki/xacro">
-  <xacro:property name="pi" value="3.14159265359" />
   <!-- Macro to add logging to a bag file. -->
   <xacro:macro name="bag_plugin_macro"
